Commit message: kedua

File: ros2_pendulum_ws/src/linear_inverted_pendulum_sim/urdf/linear_inverted_pendulum.urdf.xacro (robot description, xacro)
@@ -164,5 +164,5 @@
     <origin xyz="0 0 0" rpy="0 0 0"/>
     <axis xyz="0 1 0"/>
-    <dynamics damping="0.0003" friction="0.000001"/>
+    <dynamics damping="0.006" friction="0.00001"/>
   </joint>
   <link name="pendulum_link">

Commit message: kedua

File: ros2_pendulum_ws/src/linear_inverted_pendulum_sim/urdf/linear_inverted_pendulum.urdf.xacro (robot description, xacro)
@@ -116,5 +116,5 @@
     <origin xyz="0 0 ${pivot_z}" rpy="0 0 0"/>
     <axis xyz="1 0 0"/>
-    <limit lower="${-travel / 2.0}" upper="${travel / 2.0}" effort="100.0" velocity="3.0"/>
+    <limit lower="${-travel / 2.0}" upper="${travel / 2.0}" effort="220.0" velocity="3.0"/>
     <dynamics damping="0.02" friction="0.0005"/>
   </joint>
@@ -164,5 +164,5 @@
     <origin xyz="0 0 0" rpy="0 0 0"/>
     <axis xyz="0 1 0"/>
-    <dynamics damping="0.006" friction="0.00001"/>
+    <dynamics damping="0.05" friction="0.0005"/>
   </joint>
   <link name="pendulum_link">

Commit message: bisa tegak

File: ros2_pendulum_ws/src/linear_inverted_pendulum_sim/urdf/linear_inverted_pendulum.urdf.xacro (robot description, xacro)
@@ -116,5 +116,5 @@
     <origin xyz="0 0 ${pivot_z}" rpy="0 0 0"/>
     <axis xyz="1 0 0"/>
-    <limit lower="${-travel / 2.0}" upper="${travel / 2.0}" effort="220.0" velocity="3.0"/>
+    <limit lower="${-travel / 2.0}" upper="${travel / 2.0}" effort="360.0" velocity="4.0"/>
     <dynamics damping="0.02" friction="0.0005"/>
   </joint>
@@ -232,4 +232,7 @@
       <joint_name>cart_slider</joint_name>
     </plugin>
+    <plugin filename="gz-sim-apply-joint-force-system" name="gz::sim::systems::ApplyJointForce">
+      <joint_name>pendulum_hinge</joint_name>
+    </plugin>
   </gazebo>
 </robot>

Commit message: selesai tinggal nyempurnaiin

File: ros2_pendulum_ws/src/linear_inverted_pendulum_sim/urdf/linear_inverted_pendulum.urdf.xacro (robot description, xacro)
@@ -116,5 +116,5 @@
     <origin xyz="0 0 ${pivot_z}" rpy="0 0 0"/>
     <axis xyz="1 0 0"/>
-    <limit lower="${-travel / 2.0}" upper="${travel / 2.0}" effort="360.0" velocity="4.0"/>
+    <limit lower="${-travel / 2.0}" upper="${travel / 2.0}" effort="150.0" velocity="2.2"/>
     <dynamics damping="0.02" friction="0.0005"/>
   </joint>
